File: ESP8266_RGBA_Receiver.sch (KiCad schematic (older format))
At the start: 20 parts, among them J1 RGBAConnector, P1 ISP, Q1 PMV16XNR, Q2 PMV16XNR, Q3 PMV16XNR, Q4 PMV16XNR, SW1 SW_Push, U1 MCP1702-3302_SOT223, U2 ESP-07

Commit message: v3 as ordered on JLC PCB: ------------------------- - Replaced LED connector with Molex straddle mounted on the PCB - Moved button from GPIO0 to GPIO5 - Enlarged holes for powerinput
Parts:
- removed J1: RGBAConnector, footprint:7Wire_Solder, symbol MyLib:RGBAConnector
- added J1: Vin_Solderpad, footprint:2Wire_Solder_large, symbol MyLib:Vin_Solderpad
- added J2: Conn_02x04_Counter_Clockwise, footprint:MolexMicroFit3.0_2x8_StradleMount, symbol Connector_Generic:Conn_02x04_Counter_Clockwise
- R6: value 820R -> 560R
Connections:
- wire segments 89 -> 95
Other:
- moved on the sheet: P1, R8, SW1
Changed lines of the file:
@@
-$EndComp
-$Comp
-L MyLib:RGBAConnector J1
-U 1 1 5E697905
-P 1800 3250
-F 0 "J1" H 1833 3815 50  0000 C CNN
-F 1 "RGBAConnector" H 1833 3724 50  0000 C CNN
-F 2 "footprint:7Wire_Solder" H 2050 3700 50  0001 C CNN
-F 3 "" H 2050 3700 50  0001 C CNN
-	1    1800 3250
-	1    0    0    -1
 $EndComp
 $Comp
@@
 	1    0    0    -1
 $EndComp
-Wire Wire Line
-	2050 3450 2150 3450
 $Comp
 L Device:C C1
@@
 	4800 3450 4800 3350
 Connection ~ 2300 3950
-Wire Wire Line
-	2050 3350 2150 3350
-Wire Wire Line
-	2150 3350 2150 3450
-Connection ~ 2150 3450
-Wire Wire Line
-	2150 3450 2800 3450
 $Comp
 L power:GND #PWR014
@@
 P 6550 2750
 F 0 "R6" H 6491 2704 50  0000 R CNN
-F 1 "820R" H 6491 2795 50  0000 R CNN
+F 1 "560R" H 6491 2795 50  0000 R CNN
 F 2 "Resistor_SMD:R_0603_1608Metric" H 6550 2750 50  0001 C CNN
 F 3 "~" H 6550 2750 50  0001 C CNN
@@
 	8750 2550 9100 2550
 Wire Wire Line
-	8750 2650 9100 2650
+	8750 2650 10000 2650
 Wire Wire Line
 	8750 2750 9100 2750
@@
 L POGO_ISP:ISP P1
 U 1 1 5E6831F0
-P 3750 1900
-F 0 "P1" H 3750 2215 50  0000 C CNN
-F 1 "ISP" H 3750 2124 50  0000 C CNN
-F 2 "footprint:POGO_ISP" H 3750 700 50  0001 C CNN
-F 3 "" H 3750 700 50  0000 C CNN
-	1    3750 1900
-	1    0    0    -1
-$EndComp
-Wire Wire Line
-	4100 1800 4150 1800
-Wire Wire Line
-	4100 1900 4350 1900
-Wire Wire Line
-	4100 2000 4150 2000
-Wire Wire Line
-	3400 1800 3150 1800
-Wire Wire Line
-	3400 1900 3150 1900
-Wire Wire Line
-	3400 2000 3150 2000
+P 4250 1950
+F 0 "P1" H 4250 2265 50  0000 C CNN
+F 1 "ISP" H 4250 2174 50  0000 C CNN
+F 2 "footprint:POGO_ISP" H 4250 750 50  0001 C CNN
+F 3 "" H 4250 750 50  0000 C CNN
+	1    4250 1950
+	1    0    0    -1
+$EndComp
+Wire Wire Line
+	4600 1850 4650 1850
+Wire Wire Line
+	4600 1950 4850 1950
+Wire Wire Line
+	4600 2050 4650 2050
+Wire Wire Line
+	3900 1850 3650 1850
+Wire Wire Line
+	3900 1950 3650 1950
+Wire Wire Line
+	3900 2050 3650 2050
 $Comp
 L power:+3.3V #PWR05
 U 1 1 5E6895D5
-P 4150 1800
-F 0 "#PWR05" H 4150 1650 50  0001 C CNN
-F 1 "+3.3V" H 4165 1973 50  0000 C CNN
-F 2 "" H 4150 1800 50  0001 C CNN
-F 3 "" H 4150 1800 50  0001 C CNN
-	1    4150 1800
+P 4650 1850
+F 0 "#PWR05" H 4650 1700 50  0001 C CNN
+F 1 "+3.3V" H 4665 2023 50  0000 C CNN
+F 2 "" H 4650 1850 50  0001 C CNN
+F 3 "" H 4650 1850 50  0001 C CNN
+	1    4650 1850
 	1    0    0    -1
 $EndComp
@@
 L power:GND #PWR06
 U 1 1 5E689F65
-P 4150 2000
-F 0 "#PWR06" H 4150 1750 50  0001 C CNN
-F 1 "GND" H 4155 1827 50  0000 C CNN
-F 2 "" H 4150 2000 50  0001 C CNN
-F 3 "" H 4150 2000 50  0001 C CNN
-	1    4150 2000
-	1    0    0    -1
-$EndComp
-Text Label 3150 2000 0    50   ~ 0
+P 4650 2050
+F 0 "#PWR06" H 4650 1800 50  0001 C CNN
+F 1 "GND" H 4655 1877 50  0000 C CNN
+F 2 "" H 4650 2050 50  0001 C CNN
+F 3 "" H 4650 2050 50  0001 C CNN
+	1    4650 2050
+	1    0    0    -1
+$EndComp
+Text Label 3650 2050 0    50   ~ 0
 nRST
-Text Label 3150 1900 0    50   ~ 0
+Text Label 3650 1950 0    50   ~ 0
 GPIO0
-Text Label 3150 1800 0    50   ~ 0
+Text Label 3650 1850 0    50   ~ 0
 TXD
-Text Label 4200 1900 0    50   ~ 0
+Text Label 4700 1950 0    50   ~ 0
 RXD
 $Comp
@@
 	2150 5200 2400 5200
 Wire Wire Line
-	2050 2950 2450 2950
-Wire Wire Line
-	2050 3050 2450 3050
-Wire Wire Line
-	2050 3150 2450 3150
-Wire Wire Line
-	2050 3250 2450 3250
-Text Label 2200 2950 0    50   ~ 0
+	2300 2200 2700 2200
+Wire Wire Line
+	2300 2100 2700 2100
+Wire Wire Line
+	2300 2000 2700 2000
+Wire Wire Line
+	2300 1900 2700 1900
+Text Label 2450 2200 0    50   ~ 0
 LED_R
-Text Label 2200 3050 0    50   ~ 0
+Text Label 2450 2100 0    50   ~ 0
 LED_G
-Text Label 2200 3150 0    50   ~ 0
+Text Label 2450 2000 0    50   ~ 0
 LED_B
-Text Label 2200 3250 0    50   ~ 0
+Text Label 2450 1900 0    50   ~ 0
 LED_A
 Text Label 2200 5200 0    50   ~ 0
@@
 L Switch:SW_Push SW1
 U 1 1 5E6E3CE6
-P 10100 2350
-F 0 "SW1" V 10054 2498 50  0000 L CNN
-F 1 "SW_Push" V 10145 2498 50  0000 L CNN
-F 2 "Button_Switch_SMD:SW_SPST_PTS810" H 10100 2550 50  0001 C CNN
-F 3 "~" H 10100 2550 50  0001 C CNN
-	1    10100 2350
+P 10000 3050
+F 0 "SW1" V 9954 3198 50  0000 L CNN
+F 1 "SW_Push" V 10045 3198 50  0000 L CNN
+F 2 "Button_Switch_SMD:SW_SPST_PTS810" H 10000 3250 50  0001 C CNN
+F 3 "~" H 10000 3250 50  0001 C CNN
+	1    10000 3050
 	0    1    1    0
 $EndComp
 Wire Wire Line
-	8750 2150 10100 2150
+	8750 2150 9100 2150
 $Comp
 L Device:R_Small R8
 U 1 1 5E6E7BFF
-P 10100 1950
-F 0 "R8" H 10041 1904 50  0000 R CNN
-F 1 "10k" H 10041 1995 50  0000 R CNN
-F 2 "Resistor_SMD:R_0603_1608Metric" H 10100 1950 50  0001 C CNN
-F 3 "~" H 10100 1950 50  0001 C CNN
-	1    10100 1950
+P 10000 2450
+F 0 "R8" H 9941 2404 50  0000 R CNN
+F 1 "10k" H 9941 2495 50  0000 R CNN
+F 2 "Resistor_SMD:R_0603_1608Metric" H 10000 2450 50  0001 C CNN
+F 3 "~" H 10000 2450 50  0001 C CNN
+	1    10000 2450
 	-1   0    0    1
 $EndComp
@@
 L power:+3.3V #PWR017
 U 1 1 5E6E84B7
-P 10100 1750
-F 0 "#PWR017" H 10100 1600 50  0001 C CNN
-F 1 "+3.3V" H 10115 1923 50  0000 C CNN
-F 2 "" H 10100 1750 50  0001 C CNN
-F 3 "" H 10100 1750 50  0001 C CNN
-	1    10100 1750
-	1    0    0    -1
-$EndComp
-Wire Wire Line
-	10100 1750 10100 1850
-Wire Wire Line
-	10100 2050 10100 2150
-Connection ~ 10100 2150
+P 10000 2250
+F 0 "#PWR017" H 10000 2100 50  0001 C CNN
+F 1 "+3.3V" H 10015 2423 50  0000 C CNN
+F 2 "" H 10000 2250 50  0001 C CNN
+F 3 "" H 10000 2250 50  0001 C CNN
+	1    10000 2250
+	1    0    0    -1
+$EndComp
+Wire Wire Line
+	10000 2250 10000 2350
+Wire Wire Line
+	10000 2550 10000 2650
 $Comp
 L power:GND #PWR018
 U 1 1 5E6ED2EC
-P 10100 2650
-F 0 "#PWR018" H 10100 2400 50  0001 C CNN
-F 1 "GND" H 10105 2477 50  0000 C CNN
-F 2 "" H 10100 2650 50  0001 C CNN
-F 3 "" H 10100 2650 50  0001 C CNN
-	1    10100 2650
-	1    0    0    -1
-$EndComp
-Wire Wire Line
-	10100 2550 10100 2650
+P 10000 3450
+F 0 "#PWR018" H 10000 3200 50  0001 C CNN
+F 1 "GND" H 10005 3277 50  0000 C CNN
+F 2 "" H 10000 3450 50  0001 C CNN
+F 3 "" H 10000 3450 50  0001 C CNN
+	1    10000 3450
+	1    0    0    -1
+$EndComp
+Wire Wire Line
+	10000 3250 10000 3450
 NoConn ~ 9100 2950
 NoConn ~ 9100 3150
 NoConn ~ 7600 2550
 NoConn ~ 9100 2350
+$Comp
+L MyLib:Vin_Solderpad J1
+U 1 1 5FAED97A
+P 1950 3000
+F 0 "J1" H 1883 2815 50  0000 C CNN
+F 1 "Vin_Solderpad" H 1883 2724 50  0000 C CNN
+F 2 "footprint:2Wire_Solder_large" H 1750 2750 50  0001 C CNN
+F 3 "" H 1750 2750 50  0001 C CNN
+	1    1950 3000
+	1    0    0    -1
+$EndComp
+Wire Wire Line
+	2050 3450 2800 3450
+$Comp
+L Connector_Generic:Conn_02x04_Counter_Clockwise J2
+U 1 1 5FAF6DFB
+P 2000 2000
+F 0 "J2" H 2050 2317 50  0000 C CNN
+F 1 "Conn_02x04_Counter_Clockwise" H 2050 2226 50  0000 C CNN
+F 2 "footprint:MolexMicroFit3.0_2x8_StradleMount" H 2000 2000 50  0001 C CNN
+F 3 "~" H 2000 2000 50  0001 C CNN
+	1    2000 2000
+	1    0    0    -1
+$EndComp
+Connection ~ 10000 2650
+Wire Wire Line
+	10000 2650 10000 2850
+$Comp
+L power:GND #PWR?
+U 1 1 5FB01725
+P 1650 2300
+F 0 "#PWR?" H 1650 2050 50  0001 C CNN
+F 1 "GND" H 1655 2127 50  0000 C CNN
+F 2 "" H 1650 2300 50  0001 C CNN
+F 3 "" H 1650 2300 50  0001 C CNN
+	1    1650 2300
+	1    0    0    -1
+$EndComp
+Wire Wire Line
+	1800 1900 1650 1900
+Wire Wire Line
+	1650 1900 1650 2000
+Wire Wire Line
+	1800 2000 1650 2000
+Connection ~ 1650 2000
+Wire Wire Line
+	1650 2000 1650 2100
+Wire Wire Line
+	1800 2100 1650 2100
+Connection ~ 1650 2100
+Wire Wire Line
+	1650 2100 1650 2200
+Wire Wire Line
+	1800 2200 1650 2200
+Connection ~ 1650 2200
+Wire Wire Line
+	1650 2200 1650 2300
 $EndSCHEMATC
