File: _autosave-ESP8266_RGBA_Receiver.kicad_pcb (KiCad board)
At the start: 2 copper layers, 25.4 x 28.8 mm, 21 parts, among them J1 Vin_Solderpad, J2 Conn_02x04_Counter_Clockwise, P1 ISP, Q1 PMV16XNR, Q2 PMV16XNR, Q3 PMV16XNR, Q4 PMV16XNR, SW1 SW_Push, U1 MCP1702-3302_SOT223, U2 ESP-07

Commit message: v3 as ordered on JLC PCB: ------------------------- - Replaced LED connector with Molex straddle mounted on the PCB - Moved button from GPIO0 to GPIO5 - Enlarged holes for powerinput
Other:
- board text added: "RGBWController v3"
- board text removed: "RGBWController v2"
Changed lines of the file:
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@@
   (layers
     (0 F.Cu signal)
-    (31 B.Cu signal)
+    (31 B.Cu signal hide)
     (32 B.Adhes user hide)
     (33 F.Adhes user hide)
     (34 B.Paste user hide)
     (35 F.Paste user hide)
-    (36 B.SilkS user hide)
-    (37 F.SilkS user hide)
+    (36 B.SilkS user)
+    (37 F.SilkS user)
     (38 B.Mask user hide)
     (39 F.Mask user hide)
@@
   (module footprint:MolexMicroFit3.0_2x8_StradleMount (layer F.Cu)
     (at 91 78.5)
-    (fp_text reference J2 (at 9.5 -6.5) (layer F.SilkS)
+    (fp_text reference J2 (at -2.5 -2.7) (layer F.SilkS)
       (effects (font (size 1 1) (thickness 0.15)))
     )
@@
   (gr_arc (start 79.1718 77.2922) (end 78.105 77.2922) (angle -90) (layer Edge.Cuts) (width 0.05))
   (gr_arc (start 79.1718 50.5968) (end 79.1718 49.53) (angle -90) (layer Edge.Cuts) (width 0.05))
-  (gr_text "RGBWController v2" (at 90.17 51.562) (layer F.SilkS)
+  (gr_text "RGBWController v3" (at 90.17 51.562) (layer F.SilkS)
     (effects (font (size 0.75 0.75) (thickness 0.15)))
   )
